Commit message: sync robots with controller updates

File: configs/bruno_config/urdf/quadruped.urdf (robot description, URDF)
Before this commit: robot quadruped, 21 links, 20 joints
Joints:
- joint lf_debug_joint: origin xyz=0.138 0.04 0 rpy=0 0 0 -> xyz=0.1425 0.04 0 rpy=0 0 0
- joint lf_hip_joint: origin xyz=0.138 0.04 0.0 rpy=0 0 0 -> xyz=0.1425 0.04 0.0 rpy=0 0 0
- joint lh_debug_joint: origin xyz=-0.138 0.04 0 rpy=0 0 0 -> xyz=-0.1425 0.04 0 rpy=0 0 0
- joint lh_hip_joint: origin xyz=-0.138 0.04 0.0 rpy=0 0 0 -> xyz=-0.1425 0.04 0.0 rpy=0 0 0
- joint rf_debug_joint: origin xyz=0.138 -0.04 0 rpy=0 0 0 -> xyz=0.1425 -0.04 0 rpy=0 0 0
- joint rf_hip_joint: origin xyz=0.138 -0.04 0.0 rpy=0 0 0 -> xyz=0.1425 -0.04 0.0 rpy=0 0 0
- joint rh_debug_joint: origin xyz=-0.138 -0.04 0 rpy=0 0 0 -> xyz=-0.1425 -0.04 0 rpy=0 0 0
- joint rh_hip_joint: origin xyz=-0.138 -0.04 0.0 rpy=0 0 0 -> xyz=-0.1425 -0.04 0.0 rpy=0 0 0
